File: micrcontrolador.kicad_sch (KiCad schematic)
At the start: 10 parts, among them U3 PIC24HJ128GP502, Y1 8MHz

Commit message: cristall
Changed lines of the file:
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@@
 	(wire
 		(pts
-			(xy 143.51 133.35) (xy 143.51 171.45)
+			(xy 143.51 133.35) (xy 143.51 140.97)
 		)
 		(stroke
@@
 	(global_label "V_regulador2"
 		(shape input)
-		(at 143.51 171.45 270)
+		(at 143.51 140.97 270)
 		(fields_autoplaced yes)
 		(effects
@@
 		)
 		(property "Intersheetrefs" "${INTERSHEET_REFS}"
-			(at 143.51 187.2481 90)
+			(at 143.51 156.7681 90)
 			(effects
 				(font
