File: maleter_EDD_dc_CampaneraMireia_MartinAlba.kicad_pcb (KiCad board)
At the start: 2 copper layers, 49 parts, among them J1 Conn_01x02_Pin, J2 DE9_Pins, J3 DE9_Pins, J4 Conn_01x05_Pin, M1 Motor_DC_ALT, Q1 IRLZ44N, SW1 SW_DPST_x2, SW3 SW_DPST_x2, SW4 SW_SPDT, U1 LM2596S-5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

Commit message: Ultima versio projecte
Parts:
- added C16: 0.1uF, Capacitor_SMD:C_0201_0603Metric, F.Cu at (185.6, 39.1)
- added D3: LED, LED_SMD:LED_0201_0603Metric, F.Cu at (185.8, 44.3)
- added R14: 15k, Resistor_SMD:R_0201_0603Metric, F.Cu at (185.6, 40.8)
- added R16: 150, Resistor_SMD:R_0201_0603Metric, F.Cu at (185.6, 42.6)
- added SW2: SW_DPST_x2, Button_Switch_SMD:SW_DIP_SPSTx02_Slide_6.7x6.64mm_W6.73mm_P2.54mm_LowProfile_JPin, F.Cu at (179.1, 42.4)
- added SW4: SW_DPST_x2, Button_Switch_SMD:SW_DIP_SPSTx02_Slide_6.7x6.64mm_W6.73mm_P2.54mm_LowProfile_JPin, F.Cu at (179.1, 50.7)
- J2, J3: footprint Connector_Dsub:DSUB-9_Pins_Vertical_P2.77x2.84mm -> Connector_Dsub:DSUB-9_Pins_Horizontal_P2.77x2.84mm_EdgePinOffset9.40mm
Connections:
- net Net-(U4-CANH) renamed /POWER & COMMUNICATIONS/CANH
- net Net-(U4-CANL) renamed /POWER & COMMUNICATIONS/CANL
- R1 pad 1: SCL -> 3.3V
- R1 pad 2: Net-(U3-TCK/SCL1/RP8/CN22/PMD4/RB8) -> SCL
- R2 pad 1: SDA -> 3.3V
- R2 pad 2: Net-(U3-TDO/SDA1/RP9/CN21/PMD3/RB9) -> SDA
- U3 pad 17: Net-(U3-TCK/SCL1/RP8/CN22/PMD4/RB8) -> SCL
- U3 pad 18: Net-(U3-TDO/SDA1/RP9/CN21/PMD3/RB9) -> SDA
- U3 pad 24: unconnected-(U3-AN11/RP13/CN13/PMRD/RB13-Pad24) -> Net-(D3-A)
- U5 pad 4: unconnected-(U5-ILIM-Pad4) -> Net-(U5-ILIM)

Commit message: layout v1
Parts:
- removed SW4: SW_DPST_x2, Button_Switch_SMD:SW_DIP_SPSTx02_Slide_6.7x6.64mm_W6.73mm_P2.54mm_LowProfile_JPin
- removed SW4: SW_SPDT, Button_Switch_THT:SW_XKB_DM1-16UP-1
- removed U6: INA180A1, Package_TO_SOT_SMD:SOT-23-5
- added C17: 0.1uF, Capacitor_SMD:C_0201_0603Metric, F.Cu at (77.3, 25.6)
- added FB1: FerriteBead, Inductor_SMD:L_0201_0603Metric, F.Cu at (77.3, 27.4)
- added R15: 6k8, Resistor_SMD:R_1206_3216Metric, F.Cu at (119.2, 127.0)
- added R17: 10k, Resistor_SMD:R_1206_3216Metric, F.Cu at (119.5, 130.8)
- added SW5: SW_Push, Button_Switch_THT:SW_PUSH_6mm, F.Cu at (75.7, 44.8)
- added U9: LM358, Package_SO:SOIC-8_5.3x6.2mm_P1.27mm, F.Cu at (117.2, 121.8)
- moved D3 144.3 mm to (43.3, 66.8)
- moved Q1 119.7 mm to (33.5, 65.7)
- moved SW2 111.4 mm to (68.4, 30.3)
- moved U7 108.6 mm to (45.2, 63.9)
- moved R14 105.1 mm to (125.1, 126.8)
- moved R16 104.7 mm to (82.2, 25.6)
- moved C16 103.5 mm to (130.6, 126.8)
- moved C5 100.1 mm to (74.9, 18.6)
- moved C6 100.1 mm to (74.9, 20.4)
- moved C7 100.1 mm to (74.9, 22.1)
- moved C8 100.1 mm to (74.9, 23.9)
- moved C14 99.8 mm to (77.3, 22.1)
- moved C15 99.8 mm to (77.3, 23.9)
- moved J4 99.5 mm to (65.5, 56.2)
- moved R11 98.9 mm to (82.2, 20.4)
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Connections:
- net /POWER & COMMUNICATIONS/5V renamed /ALIMENTACIO I MOTOR/5V
- net /POWER & COMMUNICATIONS/CANH renamed /CONTROL UNIT/CANH
- net /POWER & COMMUNICATIONS/CANL renamed /CONTROL UNIT/CANL
- C7 pad 1: 3.3V -> Net-(U3-AVDD)
- U3 pad 19: GND -> (no net)
- U3 pad 28: 3.3V -> Net-(U3-AVDD)
Other:
- board text added: "${REFERENCE}"

Commit message: layout v2
Parts:
- moved J3 136.1 mm to (164.0, 100.7), turned to 180 degrees
- moved Q1 133.4 mm to (154.9, 121.0)
- moved C12 123.4 mm to (155.3, 114.2)
- moved R9 123.2 mm to (156.7, 116.8)
- moved C10 119.7 mm to (157.2, 114.2)
- moved C11 119.6 mm to (158.9, 114.2)
- moved R6 118.1 mm to (155.0, 116.8)
- moved J2 117.6 mm to (116.2, 110.7), turned to -90 degrees
- moved U7 108.3 mm to (147.5, 99.6), turned to -90 degrees
- moved U8 107.2 mm to (158.8, 107.5), turned to 90 degrees
- moved C6 105.1 mm to (138.9, 103.8)
- moved R2 104.8 mm to (145.0, 100.6), turned to 90 degrees
- moved D3 102.8 mm to (142.0, 95.6), turned to 180 degrees
- moved C9 102.7 mm to (127.2, 114.0), turned to -90 degrees
- moved C13 101.7 mm to (135.6, 103.8)
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Other:
- board outline added: 80.8 x 76.5 mm

Commit message: lay out
Parts:
- added ?: , , F.Cu at (175.8, 83.8)
- added ?: , , F.Cu at (97.2, 146.2)
- added ?: , , F.Cu at (98.0, 84.2)
- added ?: , , F.Cu at (175.5, 146.2)
- added REF**: MountingHole_2.2mm_M2_DIN965_Pad, MountingHole:MountingHole_2.2mm_M2_DIN965_Pad, F.Cu at (175.5, 146.2)
- added REF**: MountingHole_2.2mm_M2_DIN965_Pad, MountingHole:MountingHole_2.2mm_M2_DIN965_Pad, F.Cu at (175.8, 83.8)
- added REF**: MountingHole_2.2mm_M2_DIN965_Pad, MountingHole:MountingHole_2.2mm_M2_DIN965_Pad, F.Cu at (98.0, 84.2)
- added REF**: MountingHole_2.2mm_M2_DIN965_Pad, MountingHole:MountingHole_2.2mm_M2_DIN965_Pad, F.Cu at (97.2, 146.2)
- moved J1 40.1 mm to (170.0, 128.8), turned to 0 degrees
- moved F1 29.2 mm to (135.4, 146.7), turned to 90 degrees
- moved C13 22.8 mm to (144.3, 124.8)
- moved C17 22.8 mm to (146.0, 124.8)
- moved C6 22.8 mm to (147.7, 124.8)
- moved C8 22.8 mm to (150.8, 119.3)
- moved D3 22.8 mm to (150.8, 116.6)
- moved FB1 22.8 mm to (150.7, 114.1)
- moved R1 22.8 mm to (153.7, 119.9)
- moved R11 22.8 mm to (142.7, 124.8)
- moved R16 22.8 mm to (152.6, 116.6)
- moved R2 22.8 mm to (153.7, 121.6)
- moved R5 22.8 mm to (139.2, 113.8)
- moved U3 22.8 mm to (145.0, 118.2)
- moved U7 22.8 mm to (156.2, 120.6)
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Routing:
- net GND: track 0.00 -> 92.2 mm, vias 0 -> 44
- net /CONTROL UNIT/PGC: track 0.00 -> 39.0 mm
- net /CONTROL UNIT/PGD: track 0.00 -> 33.8 mm
- net 3.3V: track 0.00 -> 33.2 mm
- net MCLR: track 0.00 -> 32.1 mm
- net AntiAtrapament: track 0.00 -> 27.8 mm, vias 0 -> 2
- net Calefactor: track 0.00 -> 25.8 mm, vias 0 -> 2
- net PWM: track 0.00 -> 22.5 mm, vias 0 -> 2
- net FinalCarrera: track 0.00 -> 21.6 mm, vias 0 -> 2
- net ON/OFF: track 0.00 -> 18.8 mm, vias 0 -> 2
- net Direccio: track 0.00 -> 17.2 mm, vias 0 -> 2
- net Net-(U1-VIN): track 0.00 -> 16.3 mm
- net Net-(D1-K): track 0.00 -> 13.5 mm
- net /ALIMENTACIO I MOTOR/outamp: track 0.00 -> 13.4 mm
- net Net-(U9A-+): track 0.00 -> 12.8 mm
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- added copper zone on F.Cu, net +12V
- added copper zone on F.Cu, net +5V
- added copper zone on F.Cu, net 3.3V
- added copper zone on B.Cu, net GND
Other:
- board size 80.8 x 76.5 mm -> 85 x 68.5 mm
