File: maleter_EDD_dc_CampaneraMireia_MartinAlba.kicad_pcb (KiCad board)
At the start: 2 copper layers, 85 x 68.5 mm, 66 parts, among them J1 Conn_01x02_Pin, J2 DE9_Pins, J3 DE9_Pins, J4 Conn_01x05_Pin, M1 Motor_DC_ALT, Q1 IRLZ44N, SW1 SW_DPST_x2, SW2 SW_DPST_x2, SW3 SW_DPST_x2, SW5 SW_Push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

Commit message: Actualització projecte a classe
Parts:
- removed the ? at (175.8, 83.8)
- added J5: Conn_01x02_Pin, Connector_PinSocket_1.27mm:PinSocket_1x02_P1.27mm_Vertical, F.Cu at (174.8, 122.8)
- moved R15 13.3 mm to (155.5, 147.9)
- moved R17 12.6 mm to (155.4, 144.8), turned to 180 degrees
- moved U9 11.0 mm to (147.4, 145.3)
- moved ? 8.59 mm to (103.2, 91.0)
- moved REF** 8.59 mm to (103.2, 91.0)
- moved REF** 7.41 mm to (176.1, 91.2)
- moved ? 5.47 mm to (102.7, 146.8)
- moved REF** 5.47 mm to (102.7, 146.8)
- moved J1 5.12 mm to (175.0, 129.8)
- moved J4 4.74 mm to (143.7, 90.8)
- moved R14 4.57 mm to (145.2, 139.7)
- moved F1 3.39 mm to (132.0, 146.7), turned to 180 degrees
- moved J2 2.85 mm to (111.6, 113.2)
- moved Y1 2.50 mm to (131.0, 123.4)
- moved J3 2.42 mm to (168.6, 100.3)
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Connections:
- net Net-(D1-K) renamed /ALIMENTACIO I MOTOR/Vout
- net Net-(D3-A) renamed /CONTROL UNIT/LED
- net Net-(D3-K) renamed /CONTROL UNIT/R_LED
- net Net-(M1-+) renamed /ALIMENTACIO I MOTOR/OUT1
- net Net-(M1--) renamed /ALIMENTACIO I MOTOR/OUT2
- net Net-(U1-VIN) renamed /ALIMENTACIO I MOTOR/Vin
- net Net-(U3-AVDD) renamed /CONTROL UNIT/AVDD
- net Net-(U3-OSC1) renamed /CONTROL UNIT/OSC1
- net Net-(U3-OSC2) renamed /CONTROL UNIT/OSC2
- net Net-(U3-VCAP) renamed /CONTROL UNIT/VCAP
- net Net-(U4-Rs) renamed /CONTROL UNIT/Rs
- net Net-(U5-ILIM) renamed /ALIMENTACIO I MOTOR/ILIM
- net Net-(U8-C1+) renamed /CONTROL UNIT/C1+
- net Net-(U8-C1-) renamed /CONTROL UNIT/C1-
- net Net-(U8-C2+) renamed /CONTROL UNIT/C2+
- net Net-(U8-C2-) renamed /CONTROL UNIT/C2-
- net Net-(U8-VS+) renamed /CONTROL UNIT/VS+
- net Net-(U8-VS-) renamed /CONTROL UNIT/VS-
- C5 pad 1: Net-(C5-Pad1) -> MCLR
- Q1 pad 1: Net-(Q1-G) -> CV
- Q1 pad 2: +12V -> /CONTROL UNIT/Conn_calefactor
- R10 pad 2: Net-(U9A-+) -> /ALIMENTACIO I MOTOR/PGND
- R4 pad 2: Net-(C5-Pad1) -> MCLR
- R5 pad 1: Net-(C5-Pad1) -> MCLR
- R6 pad 2: Net-(Q1-G) -> CV
- R9 pad 1: Net-(Q1-G) -> CV
- SW5 pad 2: Net-(C5-Pad1) -> MCLR
- U3 pad 11: unconnected-(U3-RB4-Pad11) -> RX_CAN
- U3 pad 14: unconnected-(U3-RB5-Pad14) -> TX_CAN
- U3 pad 25: unconnected-(U3-RB14-Pad25) -> TX_USART
- U3 pad 26: unconnected-(U3-RB15-Pad26) -> RX_USART
- U5 pad 1: Net-(U9A-+) -> GND
- U5 pad 7: Net-(U9A-+) -> /ALIMENTACIO I MOTOR/PGND
- U5 pad 9: Net-(U9A-+) -> GND
- U9 pad 3: Net-(U9A-+) -> /ALIMENTACIO I MOTOR/PGND
Routing:
- net /CONTROL UNIT/PGC: track 39.0 -> 5.28 mm
- net /CONTROL UNIT/PGD: track 33.8 -> 4.58 mm
- net 3.3V: track 33.2 -> 6.73 mm
- net PWM: track 22.5 -> 0.89 mm, vias 2 -> 0
- net RX_CAN: track 0.00 -> 21.3 mm, vias 0 -> 2
- net TX_USART: track 0.00 -> 21.2 mm, vias 0 -> 2
- net TX_CAN: track 0.00 -> 19.7 mm, vias 0 -> 2
- net RX_USART: track 0.00 -> 18.5 mm, vias 0 -> 2
- net Direccio: track 17.2 -> 0.00 mm, vias 2 -> 0
- net GND: track 92.2 -> 78.8 mm, vias 44 -> 43
- net /ALIMENTACIO I MOTOR/PGND: track 0.00 -> 13.4 mm, vias 0 -> 2
- net Net-(U9A-+): track 12.8 -> 0.00 mm
- net /CONTROL UNIT/Conn_calefactor: track 0.00 -> 10.4 mm
- net Net-(C5-Pad1): track 10.0 -> 0.00 mm, vias 2 -> 0
- net /ALIMENTACIO I MOTOR/outamp: track 13.4 -> 3.43 mm
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- added copper zone on F.Cu, net GND
Other:
- board size 85 x 68.5 mm -> 80 x 62.2 mm
- board text added: "Maleter EDD dc Mireia Campanera Alba Martín"

Commit message: hola
Routing:
- net /CONTROL UNIT/PGC: track 5.28 -> 41.9 mm
- net /CONTROL UNIT/PGD: track 4.58 -> 39.8 mm
- net PWM: track 0.89 -> 22.9 mm
- net Direccio: track 0.00 -> 21.4 mm
- net /CONTROL UNIT/OSC2: track 12.3 -> 17.8 mm, vias 2 -> 0
- net GND: track 78.8 -> 82.1 mm, vias 43 -> 46
- net MCLR: track 37.1 -> 39.1 mm
- net AntiAtrapament: track 32.9 -> 33.7 mm
- net FinalCarrera: track 21.6 -> 20.8 mm, vias 2 -> 0
- net RX_CAN: track 21.3 -> 20.9 mm, vias 2 -> 0
- net TX_CAN: track 19.7 -> 19.8 mm, vias 2 -> 0
- net Calefactor: vias 2 -> 0
- net ON/OFF: vias 2 -> 0
- net /CONTROL UNIT/OSC1: vias 2 -> 0

Commit message: Millores profe pcb
Parts:
- moved C10 11.3 mm to (170.6, 109.5), turned to -90 degrees
- moved ? 1.45 mm to (103.2, 92.5)
- moved REF** 1.45 mm to (103.2, 92.5)
- moved REF** 1.00 mm to (176.0, 92.2)
Routing:
- net /CONTROL UNIT/VS+: track 5.38 -> 12.6 mm, vias 2 -> 0
- net TX_CAN: track 19.8 -> 27.0 mm
- net GND: track 82.1 -> 87.4 mm, vias 46 -> 83
- net /CONTROL UNIT/OSC2: track 17.8 -> 13.9 mm
- net Direccio: track 21.4 -> 18.2 mm, vias 0 -> 2
- net PWM: track 22.9 -> 24.5 mm
- net RX_CAN: track 20.9 -> 22.2 mm, vias 0 -> 2
- net /CONTROL UNIT/VS-: track 6.63 -> 7.56 mm
- net /CONTROL UNIT/C2-: track 3.57 -> 4.43 mm
- net AntiAtrapament: track 33.7 -> 34.3 mm
- net TX_USART: track 21.2 -> 21.6 mm, vias 2 -> 0
- net RX_USART: track 18.5 -> 18.4 mm, vias 2 -> 0

Commit message: mes canvis
Routing:
- net /CONTROL UNIT/CANH: track 7.30 -> 10.1 mm
- net MCLR: track 39.1 -> 38.3 mm
- net GND: track 87.4 -> 88.0 mm, vias 83 -> 85
Changed lines of the file:
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@@
+	)
+	(segment
+		(start 123.475 116.69)
+		(end 123.45 116.665)
+		(width 0.2)
+		(layer "F.Cu")
+		(net 2)
 	)
 	(segment
@@
 	)
 	(segment
+		(start 121.835 117.135)
+		(end 121.8 117.1)
+		(width 0.2)
+		(layer "F.Cu")
+		(net 2)
+	)
+	(segment
 		(start 126 117.07)
 		(end 125.32 117.07)
@@
 	)
 	(segment
-		(start 123.475 117.135)
-		(end 125.115 117.135)
-		(width 0.2)
-		(layer "F.Cu")
-		(net 2)
-	)
-	(segment
 		(start 126.68 117.07)
 		(end 126.75 117)
@@
 	)
 	(segment
+		(start 123.475 117.135)
+		(end 123.475 116.69)
+		(width 0.2)
+		(layer "F.Cu")
+		(net 2)
+	)
+	(segment
 		(start 144.665 124.75)
 		(end 144.665 124.085)
@@
 	)
 	(segment
+		(start 123.475 117.135)
+		(end 121.835 117.135)
+		(width 0.2)
+		(layer "F.Cu")
+		(net 2)
+	)
+	(segment
 		(start 109.25 132.5)
 		(end 109.18 132.57)
@@
 	)
 	(via
+		(at 123.45 116.665)
+		(size 0.6)
+		(drill 0.3)
+		(layers "F.Cu" "B.Cu")
+		(net 2)
+	)
+	(via
 		(at 136.6 123.25)
 		(size 0.6)
@@
 	(via
 		(at 130.25 127.6)
+		(size 0.6)
+		(drill 0.3)
+		(layers "F.Cu" "B.Cu")
+		(net 2)
+	)
+	(via
+		(at 121.8 117.1)
 		(size 0.6)
 		(drill 0.3)
@@
 	)
 	(segment
-		(start 142.743777 92.150769)
-		(end 142.743777 91.03338)
-		(width 0.2)
-		(layer "F.Cu")
-		(net 23)
-	)
-	(segment
 		(start 147.029978 104.339892)
 		(end 151.001 100.36887)
@@
 	)
 	(segment
+		(start 148.5 118.575)
+		(end 147.550001 118.575)
+		(width 0.2)
+		(layer "F.Cu")
+		(net 23)
+	)
+	(segment
+		(start 151.001 96.161108)
+		(end 147.780784 92.940892)
+		(width 0.2)
+		(layer "F.Cu")
+		(net 23)
+	)
+	(segment
+		(start 144.5 104.339892)
+		(end 147.029978 104.339892)
+		(width 0.2)
+		(layer "F.Cu")
+		(net 23)
+	)
+	(segment
+		(start 147.780784 92.940892)
+		(end 143.5339 92.940892)
+		(width 0.2)
+		(layer "F.Cu")
+		(net 23)
+	)
+	(segment
+		(start 142.43 91.836992)
+		(end 142.43 90.75)
+		(width 0.2)
+		(layer "F.Cu")
+		(net 23)
+	)
+	(segment
 		(start 147.550001 118.575)
 		(end 144.5 115.524999)
@@
 	)
 	(segment
-		(start 148.5 118.575)
-		(end 147.550001 118.575)
-		(width 0.2)
-		(layer "F.Cu")
-		(net 23)
-	)
-	(segment
-		(start 151.001 96.161108)
-		(end 147.780784 92.940892)
-		(width 0.2)
-		(layer "F.Cu")
-		(net 23)
-	)
-	(segment
-		(start 147.780784 92.940892)
-		(end 143.5339 92.940892)
-		(width 0.2)
-		(layer "F.Cu")
-		(net 23)
-	)
-	(segment
-		(start 144.5 104.339892)
-		(end 147.029978 104.339892)
-		(width 0.2)
-		(layer "F.Cu")
-		(net 23)
-	)
-	(segment
 		(start 143.5339 92.940892)
-		(end 142.743777 92.150769)
+		(end 142.43 91.836992)
 		(width 0.2)
 		(layer "F.Cu")
@@
 	)
 	(segment
+		(start 138.62 92.62)
+		(end 138.62 90.75)
+		(width 0.2)
+		(layer "F.Cu")
+		(net 25)
+	)
+	(segment
 		(start 148.5 100)
 		(end 150.43 100)
@@
 	)
 	(segment
-		(start 142.64 90.55)
-		(end 139.75 93.75)
-		(width 0.2)
-		(layer "F.Cu")
-		(net 25)
-	)
-	(segment
 		(start 140.699 113.224)
 		(end 141.5 114.025)
@@
 	)
 	(segment
+		(start 139.75 93.75)
+		(end 138.62 92.62)
+		(width 0.2)
+		(layer "F.Cu")
+		(net 25)
+	)
+	(segment
 		(start 140.04239 99.75)
 		(end 140.699 113.224)
@@
 	)
 	(segment
-		(start 116.205 117.365)
-		(end 111.585331 117.365)
+		(start 116.75 116.82)
+		(end 116.205 117.365)
 		(width 0.2)
 		(layer "F.Cu")
@@
 	)
 	(segment
-		(start 116.75 116.82)
-		(end 116.205 117.365)
-		(width 0.2)
-		(layer "F.Cu")
+		(start 116.205 117.365)
+		(end 108.735331 117.365)
+		(width 0.2)
+		(layer "F.Cu")

Commit message: Canvis pcb classe
Parts:
- added TP1: TestPoint, TestPoint:TestPoint_Pad_D1.0mm, F.Cu at (171.7, 129.3)
- added TP10: TestPoint, TestPoint:TestPoint_Pad_D1.0mm, F.Cu at (115.2, 118.5)
- added TP11: TestPoint, TestPoint:TestPoint_Pad_D1.0mm, F.Cu at (114.1, 115.8)
- added TP12: TestPoint, TestPoint:TestPoint_Pad_D1.0mm, F.Cu at (160.9, 128.0)
- added TP13: TestPoint, TestPoint:TestPoint_Pad_D1.0mm, F.Cu at (171.7, 120.9)
- added TP14: TestPoint, TestPoint:TestPoint_Pad_D1.0mm, F.Cu at (163.3, 128.0)
- added TP15: TestPoint, TestPoint:TestPoint_Pad_D1.0mm, F.Cu at (142.9, 135.8)
- added TP16: TestPoint, TestPoint:TestPoint_Pad_D1.0mm, F.Cu at (145.8, 133.1)
- added TP17: TestPoint, TestPoint:TestPoint_Pad_D1.0mm, F.Cu at (154.0, 121.1)
- added TP18: TestPoint, TestPoint:TestPoint_Pad_D1.0mm, F.Cu at (151.3, 122.4)
- added TP2: TestPoint, TestPoint:TestPoint_Pad_D1.0mm, F.Cu at (171.7, 131.6)
- added TP3: TestPoint, TestPoint:TestPoint_Pad_D1.0mm, F.Cu at (123.8, 139.3)
- added TP4: TestPoint, TestPoint:TestPoint_Pad_D1.0mm, F.Cu at (123.7, 135.9)
- added TP5: TestPoint, TestPoint:TestPoint_Pad_D1.0mm, F.Cu at (110.0, 129.4)
- added TP6: TestPoint, TestPoint:TestPoint_Pad_D1.0mm, F.Cu at (110.0, 126.7)
- added TP7: TestPoint, TestPoint:TestPoint_Pad_D1.0mm, F.Cu at (140.6, 110.5)
- added TP8: TestPoint, TestPoint:TestPoint_Pad_D1.0mm, F.Cu at (154.9, 115.0)
- added TP9: TestPoint, TestPoint:TestPoint_Pad_D1.0mm, F.Cu at (153.2, 114.0)
- moved C13 25.1 mm to (158.4, 104.0)
- moved R11 14.0 mm to (156.3, 121.7), turned to 90 degrees
- moved C17 13.0 mm to (149.9, 112.3), turned to 180 degrees
- moved C6 8.75 mm to (139.4, 122.1), turned to 180 degrees
- moved U7 5.86 mm to (155.1, 126.3), turned to 180 degrees
- moved R1 4.90 mm to (156.6, 123.9)
- moved L1 2.59 mm to (128.9, 134.3)
- moved R2 2.57 mm to (155.0, 123.8), turned to -90 degrees
- moved C14 1.79 mm to (135.5, 116.7)
- moved C15 1.79 mm to (135.8, 121.5)
- moved Y1 1.79 mm to (131.3, 121.7)
- moved C7 1.71 mm to (150.2, 114.3), turned to -90 degrees
- moved C9 1.36 mm to (126.5, 115.5)
- moved FB1 1.26 mm to (149.8, 113.1), turned to 0 degrees
- moved C8 0.40 mm to (150.6, 119.0), turned to -90 degrees
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Connections:
- net /CONTROL UNIT/CANH renamed /CONTROL UNIT/CAN+
- net /CONTROL UNIT/CANL renamed /CONTROL UNIT/CAN-
Routing:
- net RX_CAN: track 22.2 -> 32.6 mm, vias 2 -> 0
- net SCL: track 1.92 -> 11.0 mm, vias 0 -> 2
- net SDA: track 2.05 -> 10.8 mm
- net /ALIMENTACIO I MOTOR/outamp: track 3.43 -> 12.0 mm
- net +12V: track 2.25 -> 9.72 mm
- net /CONTROL UNIT/PGC: track 41.9 -> 36.6 mm
- net /ALIMENTACIO I MOTOR/5V: track 0.00 -> 4.27 mm
- net /CONTROL UNIT/OSC2: track 13.9 -> 10.2 mm
- net 3.3V: track 6.73 -> 3.22 mm
- net /CONTROL UNIT/Conn_calefactor: track 10.4 -> 13.9 mm
- net CV: track 5.51 -> 8.87 mm
- net /CONTROL UNIT/CAN-: track 7.16 -> 9.94 mm
- net /ALIMENTACIO I MOTOR/Vout: track 13.5 -> 16.3 mm
- net /CONTROL UNIT/CAN+: track 10.1 -> 12.3 mm
- net TX_CAN: track 27.0 -> 28.7 mm
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- added copper zone on F.Cu, net /ALIMENTACIO I MOTOR/5V
- removed copper zone on F.Cu, net +5V

Commit message: actualizacio placa drl
Parts:
- moved C16 0.91 mm to (157.2, 140.5)
Connections:
- net /ALIMENTACIO I MOTOR/5V renamed /ALIMENTACIO I MOTOR/+5V
Routing:
- net CV: track 8.87 -> 33.1 mm, vias 0 -> 2
- net GND: track 87.6 -> 103.0 mm, vias 83 -> 94
- net 3.3V: track 3.22 -> 7.70 mm
- net +12V: track 9.72 -> 7.54 mm
- net MCLR: track 38.3 -> 38.9 mm
Other:
- rule pad_to_mask_clearance: 0 -> 0.05
- board text removed: "${REFERENCE}"

Commit message: casi esquematic acabat
Parts:
- moved J5 36.4 mm to (148.2, 147.6), turned to -90 degrees
- moved TP13 33.8 mm to (150.9, 147.6)
- moved C2 33.6 mm to (108.8, 100.5), turned to 90 degrees
- moved Q1 26.6 mm to (143.6, 144.0)
- moved R6 26.6 mm to (143.7, 139.7)
- moved R9 26.6 mm to (145.4, 139.7)
- moved TP12 26.6 mm to (142.0, 146.7)
- moved TP14 26.5 mm to (144.7, 146.8)
- moved TP15 25.4 mm to (166.2, 146.0), turned to 90 degrees
- moved R14 25.3 mm to (170.1, 143.8), turned to -90 degrees
- moved U2 25.1 mm to (108.5, 106.9), turned to 90 degrees
- moved J1 23.2 mm to (160.5, 147.9), turned to -90 degrees
- moved TP16 20.4 mm to (163.5, 143.1), turned to 90 degrees
- moved TP1 18.7 mm to (161.0, 144.7), turned to -90 degrees
- moved M1 18.5 mm to (171.8, 124.3), turned to 180 degrees
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Connections:
- C1 pad 1: /ALIMENTACIO I MOTOR/+5V -> +5V
- C3 pad 1: /ALIMENTACIO I MOTOR/+5V -> +5V
- L1 pad 1: /ALIMENTACIO I MOTOR/+5V -> +5V
- TP10 pad 1: /CONTROL UNIT/CAN+ -> TX_CAN
- TP11 pad 1: /CONTROL UNIT/CAN- -> RX_CAN
- TP3 pad 1: /ALIMENTACIO I MOTOR/+5V -> +5V
- U1 pad 4: /ALIMENTACIO I MOTOR/+5V -> +5V
- U2 pad 3: /ALIMENTACIO I MOTOR/+5V -> +5V
Routing:
- net GND: track 103.0 -> 49.5 mm, vias 94 -> 122
- net 3.3V: track 7.70 -> 25.9 mm
- net PWM: track 25.3 -> 43.4 mm
- net Direccio: track 17.9 -> 35.4 mm
- net /ALIMENTACIO I MOTOR/Vin: track 13.0 -> 0.00 mm
- net AntiAtrapament: track 35.6 -> 25.4 mm
- net /CONTROL UNIT/Conn_calefactor: track 13.9 -> 5.81 mm
- net RX_CAN: track 32.6 -> 24.8 mm
- net TX_CAN: track 28.7 -> 23.8 mm
- net /ALIMENTACIO I MOTOR/outamp: track 12.0 -> 16.4 mm, vias 0 -> 2
- net /ALIMENTACIO I MOTOR/Vout: track 16.3 -> 20.6 mm
- net /ALIMENTACIO I MOTOR/+5V: track 4.27 -> 0.00 mm
- net CV: track 33.1 -> 36.0 mm, vias 2 -> 0
- net /ALIMENTACIO I MOTOR/PGND: track 12.1 -> 14.8 mm
- net +12V: track 7.54 -> 5.54 mm
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- added copper zone on F.Cu, net +5V
- added copper zone on F.Cu, net /ALIMENTACIO I MOTOR/Vin
- removed copper zone on F.Cu, net /ALIMENTACIO I MOTOR/+5V
