File: ControlUnit.kicad_sch (KiCad schematic)
At the start: 40 parts, among them J2 DE9_Pins, J3 DE9_Pins, J4 Conn_01x05_Pin, Q1 IRLZ44N, SW1 SW_DPST_x2, SW2 SW_DPST_x2, SW3 SW_DPST_x2, SW5 SW_Push, U3 PIC24HJ128GP502, U4 MCP2551-I-SN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

Commit message: Actualització projecte a classe
Parts:
- added J5: Conn_01x02_Pin, Connector_PinSocket_1.27mm:PinSocket_1x02_P1.27mm_Vertical, symbol Connector:Conn_01x02_Pin
Connections:
- net +12V: now also J5.1 (Pin_1); no longer Q1.2 (D)
- net CV: now also Q1.1 (G), R6.2, R9.1
- net MCLR: now also C5.1, R4.2, R5.1, SW5.2
- net RX_CAN: now also U3.11 (RB4)
- net RX_USART: now also U3.26 (RB15)
- net TX_CAN: now also U3.14 (RB5)
- net TX_USART: now also U3.25 (RB14)
- net OSC1: now reaches C14.1, U3.9 (OSC1), Y1.2
- net C2+: now reaches C11.1, U8.4 (C2+)
- net C2-: now reaches C11.2, U8.5 (C2-)
- net C1+: now reaches C12.1, U8.1 (C1+)
- net VS+: now reaches C10.1, U8.2 (VS+)
- net C1-: now reaches C12.2, U8.3 (C1-)
- net VS-: now reaches C10.2, U8.6 (VS-)
- net AVDD: now reaches C7.1, FB1.2, U3.28 (RB7/PGD)
- net Rs: now reaches R8.1, U4.8 (Rs)
- net VCAP: now reaches C8.2, U3.20 (VCAP)
- net OSC2: now reaches C15.1, U3.10 (OSC2), Y1.1
- net LED: now reaches D3.2 (A), U3.24 (RB13)
- net R_LED: now reaches D3.1 (K), R16.1
- new net Conn_calefactor: J5.2 (Pin_2), Q1.2 (D)
- no-connect marks 27 -> 23
Other:
- moved on the sheet: R16

Commit message: Canvis pcb classe
Parts:
- added TP10, TP11, TP12, TP13, TP14, TP17, TP18, TP7, TP8, TP9: TestPoint, TestPoint:TestPoint_Pad_D1.0mm, symbol Connector:TestPoint
Connections:
- net +12V: now also TP13.1
- net CV: now also TP12.1
- net Conn_calefactor: now also TP14.1
- net MCLR: now also TP7.1
- net RX_USART: now also TP9.1
- net SCL: now also TP18.1
- net SDA: now also TP17.1
- net TX_USART: now also TP8.1
- net CANH renamed CAN+
- net CAN+: now also TP10.1
- net CANL renamed CAN-
- net CAN-: now also TP11.1

Commit message: casi esquematic acabat
Connections:
- net CAN+: no longer TP10.1
- net CAN-: no longer TP11.1
- net RX_CAN: now also TP11.1
- net TX_CAN: now also TP10.1
Other:
- moved on the sheet: TP10, TP11
Changed lines of the file:
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@@
 	)
 	(junction
+		(at 205.74 142.24)
+		(diameter 0)
+		(color 0 0 0 0)
+	)
+	(junction
 		(at 109.22 25.4)
 		(diameter 0)
@@
 	)
 	(junction
-		(at 236.22 144.78)
-		(diameter 0)
-		(color 0 0 0 0)
-	)
-	(junction
 		(at 166.37 31.75)
 		(diameter 0)
@@
 	)
 	(junction
-		(at 236.22 149.86)
-		(diameter 0)
-		(color 0 0 0 0)
-	)
-	(junction
 		(at 116.84 15.24)
 		(diameter 0)
@@
 	)
 	(junction
+		(at 198.12 144.78)
+		(diameter 0)
+		(color 0 0 0 0)
+	)
+	(junction
 		(at 45.72 53.34)
 		(diameter 0)
@@
 	(wire
 		(pts
-			(xy 236.22 144.78) (xy 238.76 144.78)
-		)
-		(stroke
-			(width 0)
-			(type default)
-		)
-	)
-	(wire
-		(pts
 			(xy 62.23 53.34) (xy 69.85 53.34)
 		)
@@
 	(wire
 		(pts
-			(xy 236.22 149.86) (xy 238.76 149.86)
-		)
-		(stroke
-			(width 0)
-			(type default)
-		)
-	)
-	(wire
-		(pts
-			(xy 232.41 149.86) (xy 236.22 149.86)
+			(xy 232.41 149.86) (xy 238.76 149.86)
 		)
 		(stroke
@@
 	(wire
 		(pts
+			(xy 198.12 144.78) (xy 207.01 144.78)
+		)
+		(stroke
+			(width 0)
+			(type default)
+		)
+	)
+	(wire
+		(pts
 			(xy 166.37 121.92) (xy 205.74 121.92)
 		)
@@
 	(wire
 		(pts
-			(xy 187.96 144.78) (xy 207.01 144.78)
+			(xy 187.96 144.78) (xy 198.12 144.78)
 		)
 		(stroke
@@
 	(wire
 		(pts
-			(xy 232.41 144.78) (xy 236.22 144.78)
+			(xy 232.41 144.78) (xy 238.76 144.78)
 		)
 		(stroke
@@
 	(wire
 		(pts
+			(xy 205.74 142.24) (xy 207.01 142.24)
+		)
+		(stroke
+			(width 0)
+			(type default)
+		)
+	)
+	(wire
+		(pts
 			(xy 198.12 130.81) (xy 203.2 130.81)
 		)
@@
 	(wire
 		(pts
-			(xy 199.39 142.24) (xy 207.01 142.24)
+			(xy 199.39 142.24) (xy 205.74 142.24)
 		)
 		(stroke
@@
 		)
 	)
+	(global_label "+5V"
+		(shape input)
+		(at 198.12 130.81 180)
+		(fields_autoplaced yes)
+		(effects
+			(font
+				(size 1.27 1.27)
+			)
+			(justify right)
+		)
+		(property "Intersheetrefs" "${INTERSHEET_REFS}"
+			(at 191.2643 130.81 0)
+			(effects
+				(font
+					(size 1.27 1.27)
+				)
+				(justify right)
+				(hide yes)
+			)
+		)
+	)
 	(global_label "3.3V"
 		(shape input)
@@
 	(symbol
 		(lib_id "Connector:TestPoint")
-		(at 236.22 144.78 0)
+		(at 205.74 142.24 0)
 		(unit 1)
 		(exclude_from_sim no)
@@
 		(fields_autoplaced yes)
 		(property "Reference" "TP10"
-			(at 238.76 140.2079 0)
+			(at 208.28 137.6679 0)
 			(effects
 				(font
@@
 		)
 		(property "Value" "TestPoint"
-			(at 238.76 142.7479 0)
+			(at 208.28 140.2079 0)
 			(effects
 				(font
@@
 		)
 		(property "Footprint" "TestPoint:TestPoint_Pad_D1.0mm"
-			(at 241.3 144.78 0)
+			(at 210.82 142.24 0)
 			(effects
 				(font
@@
 		)
 		(property "Datasheet" "~"
-			(at 241.3 144.78 0)
+			(at 210.82 142.24 0)
 			(effects
 				(font
@@
 		)
 		(property "Description" "test point"
-			(at 236.22 144.78 0)
+			(at 205.74 142.24 0)
 			(effects
 				(font
@@
 		)
 		(instances
-			(project ""
+			(project "maleter_EDD_dc_CampaneraMireia_MartinAlba"
 				(path "/c2b694d2-752b-44f8-812f-8731bb340544/81127ddb-0668-402b-863d-213dd1dac81e"
 					(reference "TP10")
@@
 	)
 	(symbol
-		(lib_id "power:+5V")
-		(at 198.12 130.81 0)
-		(unit 1)
-		(exclude_from_sim no)
-		(in_bom yes)
-		(on_board yes)
-		(dnp no)
-		(fields_autoplaced yes)
-		(property "Reference" "#PWR016"
-			(at 198.12 134.62 0)
-			(effects
-				(font
-					(size 1.27 1.27)
-				)
-				(hide yes)
-			)
-		)
-		(property "Value" "+5V"
-			(at 198.12 125.73 0)
-			(effects
-				(font
-					(size 1.27 1.27)
-				)
-			)
-		)
-		(property "Footprint" ""
-			(at 198.12 130.81 0)
-			(effects
-				(font
-					(size 1.27 1.27)
-				)
-				(hide yes)
-			)
-		)
-		(property "Datasheet" ""
-			(at 198.12 130.81 0)
-			(effects
-				(font
-					(size 1.27 1.27)
-				)
-				(hide yes)
-			)
-		)
-		(property "Description" "Power symbol creates a global label with name \"+5V\""
-			(at 198.12 130.81 0)
-			(effects
-				(font
-					(size 1.27 1.27)
-				)
-				(hide yes)
-			)
-		)
-		(pin "1"
-		)
-		(instances
-			(project "maleter_EDD_dc_CampaneraMireia_MartinAlba"
-				(path "/c2b694d2-752b-44f8-812f-8731bb340544/81127ddb-0668-402b-863d-213dd1dac81e"
-					(reference "#PWR016")
-					(unit 1)
-				)
-			)
-		)
-	)
-	(symbol
 		(lib_id "Device:R")
 		(at 157.48 31.75 90)
@@
 	(symbol
 		(lib_id "Connector:TestPoint")
-		(at 236.22 149.86 180)
+		(at 198.12 144.78 180)
 		(unit 1)
 		(exclude_from_sim no)
@@
 		(fields_autoplaced yes)
 		(property "Reference" "TP11"
-			(at 238.76 151.8919 0)
+			(at 200.66 146.8119 0)
 			(effects
 				(font
@@
 		)
 		(property "Value" "TestPoint"
-			(at 238.76 154.4319 0)
+			(at 200.66 149.3519 0)
 			(effects
 				(font
@@
 		)
 		(property "Footprint" "TestPoint:TestPoint_Pad_D1.0mm"
-			(at 231.14 149.86 0)
+			(at 193.04 144.78 0)
 			(effects
 				(font
@@
 		)
 		(property "Datasheet" "~"
-			(at 231.14 149.86 0)
+			(at 193.04 144.78 0)
 			(effects
 				(font
@@
 		)
 		(property "Description" "test point"
-			(at 236.22 149.86 0)
+			(at 198.12 144.78 0)
 			(effects
 				(font
