File: power&communications.kicad_sch (KiCad schematic)
At the start: 21 parts, among them J1 Conn_01x02_Pin, J2 DE9_Pins, J3 DE9_Pins, U1 LM2596S-5, U2 LM1117DT-3.3, U4 MCP2551-I-SN, U8 MAX3232

Commit message: Definició parcial huellas
Parts:
- C1, C10, C11, C12, C13, C2, C3, C4, C9: footprint (none) -> Capacitor_SMD:C_0201_0603Metric
- F1: footprint (none) -> Fuse:Fuse_0402_1005Metric
- L1: footprint (none) -> Inductor_SMD:L_6.3x6.3_H3
- R7, R8: footprint (none) -> Resistor_SMD:R_0201_0603Metric
Changed lines of the file:
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@@
 			)
 		)
-		(property "Footprint" ""
+		(property "Footprint" "Capacitor_SMD:C_0201_0603Metric"
 			(at 158.4452 59.69 0)
 			(effects
@@
 			)
 		)
-		(property "Footprint" ""
+		(property "Footprint" "Capacitor_SMD:C_0201_0603Metric"
 			(at 270.2052 115.57 0)
 			(effects
@@
 			)
 		)
-		(property "Footprint" ""
+		(property "Footprint" "Capacitor_SMD:C_0201_0603Metric"
 			(at 253.6952 105.41 0)
 			(effects
@@
 			)
 		)
-		(property "Footprint" ""
+		(property "Footprint" "Resistor_SMD:R_0201_0603Metric"
 			(at 83.312 111.76 90)
 			(effects
@@
 			)
 		)
-		(property "Footprint" ""
+		(property "Footprint" "Capacitor_SMD:C_0201_0603Metric"
 			(at 253.6952 118.11 0)
 			(effects
@@
 			)
 		)
-		(property "Footprint" ""
+		(property "Footprint" "Capacitor_SMD:C_0201_0603Metric"
 			(at 97.4852 52.07 0)
 			(effects
@@
 			)
 		)
-		(property "Footprint" ""
+		(property "Footprint" "Resistor_SMD:R_0201_0603Metric"
 			(at 43.942 121.92 90)
 			(effects
@@
 			)
 		)
-		(property "Footprint" ""
+		(property "Footprint" "Fuse:Fuse_0402_1005Metric"
 			(at 85.852 43.18 90)
 			(effects
@@
 			)
 		)
-		(property "Footprint" ""
+		(property "Footprint" "Capacitor_SMD:C_0201_0603Metric"
 			(at 173.6852 62.23 0)
 			(effects
@@
 			)
 		)
-		(property "Footprint" ""
+		(property "Footprint" "Inductor_SMD:L_6.3x6.3_H3"
 			(at 146.05 55.88 0)
 			(effects
@@
 			)
 		)
-		(property "Footprint" ""
+		(property "Footprint" "Capacitor_SMD:C_0201_0603Metric"
 			(at 199.0852 59.69 0)
 			(effects
@@
 			)
 		)
-		(property "Footprint" ""
+		(property "Footprint" "Capacitor_SMD:C_0201_0603Metric"
 			(at 46.6852 102.87 0)
 			(effects
@@
 			)
 		)
-		(property "Footprint" ""
+		(property "Footprint" "Capacitor_SMD:C_0201_0603Metric"
 			(at 199.0852 105.41 0)
 			(effects

Commit message: coses que falten
Parts:
- J1: footprint (none) -> Connector_PinSocket_1.27mm:PinSocket_1x02_P1.27mm_Vertical
- J2, J3: footprint (none) -> Connector_Dsub:DSUB-9_Pins_Vertical_P2.77x2.84mm
- U8: footprint (none) -> Package_SO:SOIC-16W_5.3x10.2mm_P1.27mm
Changed lines of the file:
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@@
 			)
 		)
-		(property "Footprint" ""
+		(property "Footprint" "Package_SO:SOIC-16W_5.3x10.2mm_P1.27mm"
 			(at 226.06 147.32 0)
 			(effects
@@
 			)
 		)
-		(property "Footprint" ""
+		(property "Footprint" "Connector_Dsub:DSUB-9_Pins_Vertical_P2.77x2.84mm"
 			(at 113.03 106.68 0)
 			(effects
@@
 			)
 		)
-		(property "Footprint" ""
+		(property "Footprint" "Connector_PinSocket_1.27mm:PinSocket_1x02_P1.27mm_Vertical"
 			(at 26.67 30.48 0)
 			(effects
@@
 			)
 		)
-		(property "Footprint" ""
+		(property "Footprint" "Connector_Dsub:DSUB-9_Pins_Vertical_P2.77x2.84mm"
 			(at 163.83 110.49 0)
 			(effects

Commit message: Correccions professor
Connections:
- net CANH: now reaches J2.7, R7.1, U4.7 (CANH)
- net CANL: now reaches J2.2, R7.2, U4.6 (CANL)
- no-connect marks 11 -> 17
Other:
- note added: "MIREIA CAMPANERA I ALBA MARTÍN PROJECTE MALETER EDD Comunicacions: Bus CAN, alimentació i connexió UART"
- note removed: "MIREIA CAMPANERA I ALBA MARTÍN PROJECTE MALETER EDD"
- moved on the sheet: C4
Changed lines of the file:
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@@
 		)
 	)
-	(text "MIREIA CAMPANERA I ALBA MARTÍN\nPROJECTE MALETER EDD"
+	(text "MIREIA CAMPANERA I ALBA MARTÍN\nPROJECTE MALETER EDD\nComunicacions: Bus CAN, alimentació i connexió UART"
 		(exclude_from_sim no)
 		(at 178.308 170.688 0)
@@
 	)
 	(no_connect
+		(at 171.45 107.95)
+	)
+	(no_connect
 		(at 105.41 104.14)
 	)
@@
 	)
 	(no_connect
+		(at 171.45 100.33)
+	)
+	(no_connect
 		(at 204.47 128.27)
 	)
@@
 	)
 	(no_connect
+		(at 171.45 102.87)
+	)
+	(no_connect
+		(at 171.45 115.57)
+	)
+	(no_connect
+		(at 171.45 118.11)
+	)
+	(no_connect
 		(at 49.53 114.3)
+	)
+	(no_connect
+		(at 171.45 113.03)
 	)
 	(no_connect
@@
 	(wire
 		(pts
-			(xy 96.52 44.45) (xy 96.52 38.1)
-		)
-		(stroke
-			(width 0)
-			(type default)
-		)
-	)
-	(wire
-		(pts
 			(xy 85.09 106.68) (xy 85.09 107.95)
 		)
@@
 		(pts
 			(xy 171.45 105.41) (xy 176.53 105.41)
-		)
-		(stroke
-			(width 0)
-			(type default)
-		)
-	)
-	(wire
-		(pts
-			(xy 96.52 38.1) (xy 105.41 38.1)
 		)
 		(stroke
@@
 				(size 1.27 1.27)
 				(thickness 0.1588)
+			)
+			(justify left bottom)
+		)
+	)
+	(label "CANL"
+		(at 92.71 116.84 0)
+		(effects
+			(font
+				(size 1.27 1.27)
+			)
+			(justify left bottom)
+		)
+	)
+	(label "CANH"
+		(at 91.44 106.68 0)
+		(effects
+			(font
+				(size 1.27 1.27)
 			)
 			(justify left bottom)
@@
 	(symbol
 		(lib_id "power:GND")
-		(at 105.41 38.1 0)
+		(at 96.52 59.69 0)
 		(unit 1)
 		(exclude_from_sim no)
@@
 		(fields_autoplaced yes)
 		(property "Reference" "#PWR09"
-			(at 105.41 44.45 0)
+			(at 96.52 66.04 0)
 			(effects
 				(font
@@
 		)
 		(property "Value" "GND"
-			(at 105.41 43.18 0)
-			(effects
-				(font
-					(size 1.27 1.27)
-				)
+			(at 99.06 60.9599 0)
+			(effects
+				(font
+					(size 1.27 1.27)
+				)
+				(justify left)
 			)
 		)
 		(property "Footprint" ""
-			(at 105.41 38.1 0)
+			(at 96.52 59.69 0)
 			(effects
 				(font
@@
 		)
 		(property "Datasheet" ""
-			(at 105.41 38.1 0)
+			(at 96.52 59.69 0)
 			(effects
 				(font
@@
 		)
 		(property "Description" "Power symbol creates a global label with name \"GND\" , ground"
-			(at 105.41 38.1 0)
+			(at 96.52 59.69 0)
 			(effects
 				(font
@@
 	(symbol
 		(lib_id "Device:C")
-		(at 96.52 48.26 0)
+		(at 96.52 55.88 180)
 		(unit 1)
 		(exclude_from_sim no)
@@
 		(fields_autoplaced yes)
 		(property "Reference" "C4"
-			(at 100.33 46.9899 0)
+			(at 92.71 57.1501 0)
 			(effects
 				(font
@@
 		)
 		(property "Value" "100uF"
-			(at 100.33 49.5299 0)
+			(at 92.71 54.6101 0)
 			(effects
 				(font
@@
 		)
 		(property "Footprint" "Capacitor_SMD:C_0201_0603Metric"
-			(at 97.4852 52.07 0)
+			(at 95.5548 52.07 0)
 			(effects
 				(font
@@
 		)
 		(property "Datasheet" "~"
-			(at 96.52 48.26 0)
+			(at 96.52 55.88 0)
 			(effects
 				(font
@@
 		)
 		(property "Description" "Unpolarized capacitor"
-			(at 96.52 48.26 0)
-			(effects
-				(font
+			(at 96.52 55.88 0)
+			(effects
+				(font

Commit message: Ultima versio projecte
Parts:
- removed C10, C11, C12, C13, C9: 100nF, Capacitor_SMD:C_0201_0603Metric, symbol Device:C
- removed J2, J3: DE9_Pins, Connector_Dsub:DSUB-9_Pins_Vertical_P2.77x2.84mm, symbol Connector:DE9_Pins
- removed R7: 120Ω, Resistor_SMD:R_0201_0603Metric, symbol Device:R
- removed R8: 10k, Resistor_SMD:R_0201_0603Metric, symbol Device:R
- removed U4: MCP2551-I-SN, Package_SO:SOIC-8_3.9x4.9mm_P1.27mm, symbol Interface_CAN_LIN:MCP2551-I-SN
- removed U8: MAX3232, Package_SO:SOIC-16W_5.3x10.2mm_P1.27mm, symbol Interface_UART:MAX3232
- added C16: 0.1uF, Capacitor_SMD:C_0201_0603Metric, symbol Device:C
- added M1: Motor_DC_ALT, TerminalBlock_CUI:TerminalBlock_CUI_TB007-508-02_1x02_P5.08mm_Horizontal, symbol Motor:Motor_DC_ALT
- added R10: 0.05, Resistor_SMD:R_0201_0603Metric, symbol Device:R
- added R14: 15k, Resistor_SMD:R_0201_0603Metric, symbol Device:R
- added R15: 6k8, Resistor_SMD:R_1206_3216Metric, symbol Device:R
- added R17: 10k, Resistor_SMD:R_1206_3216Metric, symbol Device:R
- added U5: DRV8871DDA, Package_SO:Texas_HTSOP-8-1EP_3.9x4.9mm_P1.27mm_EP2.95x4.9mm_Mask2.4x3.1mm_ThermalVias, symbol Driver_Motor:DRV8871DDA
- added U9: LM358, Package_SO:SOIC-8_5.3x6.2mm_P1.27mm, symbol Amplifier_Operational:LM358
Connections:
- net +12V: now also C16.2, U5.5 (VM)
- net GND: now also C16.1, R10.1, R14.2, R17.1
- new net: R10.2, U5.1 (GND), U5.7 (GND), U5.9 (GND), U9.3 (+)
- new net: R14.1, U5.4 (ILIM)
- new net: M1.1 (+), U5.6 (OUT1)
- new net: M1.2 (-), U5.8 (OUT2)
- new net AntiAtrapament: U9.6 (-), U9.7
- new net Direccio: U5.2 (IN2)
- new net PWM: U5.3 (IN1)
- new net op1neg: R15.1, R17.2, U9.2 (-)
- new net outamp: R15.2, U9.1, U9.5 (+)
- no-connect marks 17 -> 0
Other:
- note added: "Anti-atrapament"
- note added: "MIREIA CAMPANERA I ALBA MARTÍN PROJECTE MALETER EDD Alimentació i motor maleter"
- note added: "Motor del maleter"
- note removed: "BUS CAN"
- note removed: "MIREIA CAMPANERA I ALBA MARTÍN PROJECTE MALETER EDD Comunicacions: Bus CAN, alimentació i connexió UART"
- note removed: "USART"
- moved on the sheet: C1, C2, C3, C4, D1, F1, J1, L1, U1, U2

Commit message: Actualització projecte a classe
Connections:
- net GND: now also U5.1 (GND), U5.9 (PPAD)
- net PGND: now reaches R10.2, U5.7 (PGND), U9.3 (+)
- net PGND: no longer U5.1 (GND), U5.9 (GND)
- net ILIM: now reaches R14.1, U5.4 (ILIM)
- net OUT1: now reaches M1.1 (+), U5.6 (OUT1)
- net OUT2: now reaches M1.2 (-), U5.8 (OUT2)
- net Vout: now reaches D1.1 (K), L1.2, U1.2 (OUT)
- net Vin: now reaches C4.2, F1.2, U1.1 (VIN)

Commit message: Canvis pcb classe
Parts:
- added TP1, TP15, TP16, TP2, TP3, TP4, TP5, TP6: TestPoint, TestPoint:TestPoint_Pad_D1.0mm, symbol Connector:TestPoint
Connections:
- net +12V: now also TP1.1
- net 3.3V: now also TP5.1
- net 5V: now also TP3.1
- net Direccio: now also TP16.1
- net GND: now also TP2.1, TP4.1, TP6.1
- net PWM: now also TP15.1

Commit message: actualizacio placa drl
Connections:
- net 5V renamed +5V
Changed lines of the file:
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@@
 		)
 	)
-	(label "5V"
+	(label "+5V"
 		(at 203.2 102.87 0)
 		(effects

Commit message: casi esquematic acabat
Changed lines of the file:
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@@
 	)
 	(label "+5V"
-		(at 203.2 102.87 0)
+		(at 241.3 102.87 0)
 		(effects
 			(font
@@
 		)
 	)
+	(label "+5V"
+		(at 198.12 102.87 0)
+		(effects
+			(font
+				(size 1.27 1.27)
+				(thickness 0.1588)
+			)
+			(justify left bottom)
+		)
+	)
 	(label "ILIM"
 		(at 55.88 106.68 0)
@@
 		)
 	)
+	(global_label "+5V"
+		(shape input)
+		(at 219.71 102.87 90)
+		(fields_autoplaced yes)
+		(effects
+			(font
+				(size 1.27 1.27)
+			)
+			(justify left)
+		)
+		(property "Intersheetrefs" "${INTERSHEET_REFS}"
+			(at 219.71 96.0143 90)
+			(effects
+				(font
+					(size 1.27 1.27)
+				)
+				(justify left)
+				(hide yes)
+			)
+		)
+	)
